File: hardware/pcbs/MainCollar/MainCollar.kicad_pcb (KiCad board)
At the start: 2 copper layers, 57 x 97 mm, 78 parts, among them J1 SMA-EDGE, M1 Mounting_Hole, M2 Mounting_Hole, M3 Mounting_Hole, M4 Mounting_Hole, P1 USB_OTG, P2 CONN_01X05, P3 Solar1, P4 Solar2, P5 CONN_02X05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

Commit message: Switched R17 and R18 to be in correct locations
Parts:
- moved R18 1.72 mm to (57.2, 96.0)
- moved R17 1.67 mm to (55.5, 96.0)
Connections:
- U6 pad 12: Net-(R17-Pad1) -> Net-(R18-Pad1)
- U6 pad 13: Net-(R18-Pad1) -> Net-(R17-Pad1)
Routing:
- net Net-(R18-Pad1): track 5.85 -> 4.37 mm
- net Net-(R17-Pad1): track 4.37 -> 5.85 mm
Changed lines of the file:
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@@
     (links 219)
     (no_connects 1)
-    (area 30.6441 25.949599 135.100001 135.100001)
+    (area 35.924999 35.924999 93.075001 133.075001)
     (thickness 1.6)
     (drawings 23)
@@
       (effects (font (size 1 1) (thickness 0.15)))
     )
-    (fp_text value 0.1uF (at 0 1.9) (layer F.Fab)
+    (fp_text value 0.1uF (at -5.506 -0.168) (layer F.Fab)
       (effects (font (size 1 1) (thickness 0.15)))
     )
@@
       (effects (font (size 1 1) (thickness 0.15)))
     )
-    (fp_text value 10K (at 0 1.9) (layer F.Fab)
+    (fp_text value 10K (at -3.274 0.127) (layer F.Fab)
       (effects (font (size 1 1) (thickness 0.15)))
     )
@@
       (effects (font (size 1 1) (thickness 0.15)))
     )
-    (fp_text value 330 (at 0 1.9) (layer F.Fab)
+    (fp_text value 330 (at -5.133 0.037) (layer F.Fab)
       (effects (font (size 1 1) (thickness 0.15)))
     )
@@
   )
   (module Resistors_SMD:R_0603_HandSoldering (layer F.Cu)
-    (at 57.15 96.266 90)
+    (at 55.5 96 90)
     (descr "Resistor SMD 0603, hand soldering")
     (tags "resistor 0603")
@@
   )
   (module Resistors_SMD:R_0603_HandSoldering (layer F.Cu)
-    (at 55.499 96.266 90)
+    (at 57.2 96 90)
     (descr "Resistor SMD 0603, hand soldering")
     (tags "resistor 0603")
@@
       (net 2 GND))
     (pad 12 smd rect (at 1.965 0.5 180) (size 0.73 0.3) (layers F.Cu F.Paste F.Mask)
-      (net 56 "Net-(R17-Pad1)"))
-    (pad 13 smd rect (at 1.965 0 180) (size 0.73 0.3) (layers F.Cu F.Paste F.Mask)
       (net 57 "Net-(R18-Pad1)"))
+    (pad 13 smd rect (at 1.965 0 180) (size 0.73 0.3) (layers F.Cu F.Paste F.Mask)
+      (net 56 "Net-(R17-Pad1)"))
     (pad 14 smd rect (at 1.965 -0.5 180) (size 0.73 0.3) (layers F.Cu F.Paste F.Mask)
       (net 11 VBAT))
@@
   (segment (start 67.2465 81.8515) (end 67.012 81.617) (width 0.254) (layer F.Cu) (net 55))
   (segment (start 67.2465 86.2965) (end 67.2465 81.8515) (width 0.254) (layer F.Cu) (net 55))
-  (segment (start 57.15 97.366) (end 57.15 100.076) (width 0.254) (layer F.Cu) (net 56))
-  (segment (start 57.92 100.846) (end 58.487 100.846) (width 0.254) (layer F.Cu) (net 56))
-  (segment (start 57.15 100.076) (end 57.92 100.846) (width 0.254) (layer F.Cu) (net 56))
-  (segment (start 58.487 101.346) (end 57.404 101.346) (width 0.254) (layer F.Cu) (net 57))
-  (segment (start 55.499 99.441) (end 55.499 97.366) (width 0.254) (layer F.Cu) (net 57))
-  (segment (start 57.404 101.346) (end 55.499 99.441) (width 0.254) (layer F.Cu) (net 57))
+  (segment (start 58.487 101.346) (end 57.404 101.346) (width 0.254) (layer F.Cu) (net 56))
+  (segment (start 57.404 101.346) (end 55.499 99.441) (width 0.254) (layer F.Cu) (net 56))
+  (segment (start 55.499 99.441) (end 55.499 97.366) (width 0.254) (layer F.Cu) (net 56))
+  (segment (start 57.15 97.366) (end 57.15 100.076) (width 0.254) (layer F.Cu) (net 57))
+  (segment (start 57.15 100.076) (end 57.92 100.846) (width 0.254) (layer F.Cu) (net 57))
+  (segment (start 57.92 100.846) (end 58.487 100.846) (width 0.254) (layer F.Cu) (net 57))
   (segment (start 39.37 69.85) (end 37.592 69.85) (width 0.2032) (layer F.Cu) (net 64))
   (segment (start 54.991 69.977) (end 58.591 73.577) (width 0.2032) (layer F.Cu) (net 64))
